Commit message: Added crazyflie model and prepared for data logging

File: rotors_description/urdf/multirotor_base.xacro (robot description, xacro)
@@ -33,8 +33,8 @@
   <!-- Main multirotor link -->
   <xacro:macro name="multirotor_base_macro"
-    params="robot_namespace mass body_width body_height use_mesh_file mesh_file *inertia">
+    params="robot_namespace mass body_width body_height use_mesh_file mesh_file mesh_rotation_r:=0 mesh_rotation_p:=0 mesh_rotation_y:=0 *inertia">
     <link name="${robot_namespace}/base_link"></link>
     <joint name="${robot_namespace}/base_joint" type="fixed">
-      <origin xyz="0 0 0" rpy="0 0 0" />
+      <origin xyz="0 0 0" rpy="${mesh_rotation_r} ${mesh_rotation_p} ${mesh_rotation_y}" />
       <parent link="${robot_namespace}/base_link" />
       <child link="${robot_namespace}/base_link_inertia" />
@@ -47,5 +47,5 @@
       </inertial>
       <visual>
-        <origin xyz="0 0 0" rpy="0 0 0" />
+        <origin xyz="0 0 0" rpy="${mesh_rotation_r} ${mesh_rotation_p} ${mesh_rotation_y}" />
         <geometry>
           <xacro:if value="${use_mesh_file}">
@@ -58,5 +58,5 @@
       </visual>
       <collision>
-        <origin xyz="0 0 0" rpy="0 0 0" />
+        <origin xyz="0 0 0" rpy="${mesh_rotation_r} ${mesh_rotation_p} ${mesh_rotation_y}" />
         <geometry>
           <box size="${body_width} ${body_width} ${body_height}" /> <!-- [m] [m] [m] -->
