Commit message: Modified code to profile the simulation. This modification is only temporary.

File: rotors_description/urdf/component_snippets.xacro (robot description, xacro)
@@ -895,3 +895,25 @@
     </xacro:mavlink_interface_macro>
   </xacro:macro>
+  <xacro:macro name="crazyflie2_imu" params="namespace parent_link">
+    <!-- Mount an MPU-9250 IMU. -->
+    <xacro:imu_plugin_macro
+      namespace="${namespace}"
+      imu_suffix=""
+      parent_link="${parent_link}"
+      imu_topic="imu"
+      measurement_delay="0"
+      measurement_divisor="1"
+      mass_imu_sensor="0.00001"
+      gyroscope_noise_density="0.000175"
+      gyroscope_random_walk="0.0105"
+      gyroscope_bias_correlation_time="1000.00"
+      gyroscope_turn_on_bias_sigma="0.09"
+      accelerometer_noise_density="0.003"
+      accelerometer_random_walk="0.18"
+      accelerometer_bias_correlation_time="300.0"
+      accelerometer_turn_on_bias_sigma="0.588" >
+      <inertia ixx="0.00001" ixy="0.0" ixz="0.0" iyy="0.00001" iyz="0.0" izz="0.00001" />
+      <origin xyz="0 0 0" rpy="0 0 0" />
+    </xacro:imu_plugin_macro>
+  </xacro:macro>
 </robot>

File: rotors_description/urdf/multirotor_base.xacro (robot description, xacro)
@@ -60,5 +60,5 @@
         <origin xyz="0 0 0" rpy="${mesh_rotation_r} ${mesh_rotation_p} ${mesh_rotation_y}" />
         <geometry>
-          <box size="${body_width} ${body_width} ${body_height}" /> <!-- [m] [m] [m] -->
+          <box size="${body_width} ${body_width} ${body_height}" />  <!-- [m] [m] [m] -->
         </geometry>
       </collision>
